File: 02.Hardware/Battery PCBs/BATT_DISP/BATT_DISP.brd (EAGLE design)
At the start: 33.2 x 28 mm, 131 parts, among them K1 FLEX6, U1 IS31FL3731-SALS2

Commit message: Cambios revisados con David
Revision de los pcbs de la bateria.

En el DCDC se añade un diode Clamp (bat54s) en la medicion de la tension de salida.
Actualizacion de la BOM a v8.
Documentos de Cambios de versiones
Parts:
- moved R4 14.4 mm to (44.0, 16.3), turned to 0 degrees
- moved R7 10.1 mm to (34.1, 11.3)
- moved R6 9.23 mm to (14.9, 11.1), turned to 90 degrees
- moved C3 3.76 mm to (15.1, 14.4), turned to 0 degrees
- moved R2 3.35 mm to (18.0, 11.8)
- moved R3 1.12 mm to (43.8, 13.3)
- moved R1 0.93 mm to (37.6, 11.4)
- moved C1 0.64 mm to (16.4, 3.50)
- moved C5 0.60 mm to (26.4, 4.40)
- moved C4 0.50 mm to (30.2, 4.45)
- moved R8 0.34 mm to (33.0, 4.43)
Routing:
- net M_ADDR: track 21.8 -> 7.27 mm
- net M_SCL: track 75.0 -> 84.6 mm
- net N$1: track 14.4 -> 23.1 mm
- net VCC: track 82.0 -> 90.2 mm
- net M_SDA: track 61.2 -> 53.8 mm
- net M_CB4: track 52.9 -> 48.3 mm
- net S_DOWN: track 87.2 -> 83.7 mm
- net GND: track 25.9 -> 27.6 mm
- net S_UP: track 42.3 -> 43.4 mm
- net M_CB3: track 48.2 -> 48.9 mm
Other:
- board text added: "display_falcon v9-May22"
- board text removed: "sep-display_falcon_v8"
