File: 02.Hardware/Battery PCBs/BATT_DISP/BATT_DISP.sch (EAGLE design)
At the start: 131 parts, among them K1 FLEX6, U1 IS31FL3731-SALS2

Commit message: Cambios revisados con David
Revision de los pcbs de la bateria.

En el DCDC se añade un diode Clamp (bat54s) en la medicion de la tension de salida.
Actualizacion de la BOM a v8.
Documentos de Cambios de versiones
Changed lines of the file:
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@@
 </instance>
 <instance part="K1" gate="G$1" x="71.12" y="139.7" smashed="yes">
-<attribute name="VALUE" x="71.12" y="121.92" size="1.778" layer="96"/>
+<attribute name="VALUE" x="71.12" y="160.02" size="1.778" layer="96"/>
 </instance>
 <instance part="S1" gate="G$1" x="223.52" y="132.08" smashed="yes" rot="R180">

Commit message: review general antes de produccion
R1, R2 --> Cambiamos valor de pullup para dejarlo igual que  en EDCPSU
R8 --> Se corrige el valor para  dejarlo como recomienda en la nota de aplicacion. Comprobamos 4mA menos de consumo (de 21mA a 18mA)
Parts:
- R1, R2: value 10K -> 2k2
- R8: value 10K -> 20k
Changed lines of the file:
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@@
 <part name="R6" library="rcl" deviceset="R-EU_" device="R0603" value="10K"/>
 <part name="R7" library="rcl" deviceset="R-EU_" device="R0603" value="10K"/>
-<part name="R8" library="rcl" deviceset="R-EU_" device="R0603" value="10K"/>
+<part name="R8" library="rcl" deviceset="R-EU_" device="R0603" value="20k"/>
 <part name="K1" library="Flex_3mm" deviceset="FLEX6" device=""/>
 <part name="S1" library="switch momentary CK KXT311LHS" deviceset="KXT311LHS" device=""/>
@@
 <part name="C2" library="microbuilder" deviceset="CAP_CERAMIC" device="0805-NOOUTLINE" value="100n"/>
 <part name="C3" library="microbuilder" deviceset="CAP_CERAMIC" device="0805-NOOUTLINE" value="100n"/>
-<part name="R1" library="rcl" deviceset="R-EU_" device="R0603" value="10K"/>
-<part name="R2" library="rcl" deviceset="R-EU_" device="R0603" value="10K"/>
+<part name="R1" library="rcl" deviceset="R-EU_" device="R0603" value="2k2"/>
+<part name="R2" library="rcl" deviceset="R-EU_" device="R0603" value="2k2"/>
 <part name="P+2" library="microbuilder" deviceset="VCC" device=""/>
 <part name="P+3" library="microbuilder" deviceset="VCC" device=""/>
