File: 02.HARDWARE/V2-ROVER-1K/01.PCB/BATT_CPU/BATT_CPU.sch (EAGLE design)
At the start: 68 parts, among them J1 2314820-6, K3 FLEX_CONN, K4 FLEX6, K5 FLEX8, U1 ATSAMD21G18_QFN, U2 TPS78230DDCR, U3 TPS78230DDCR, U5 MAX9062EUK+T, U6 MAX9062EUK+T, U7 MCP6071T-E/OT, U8 SN74LVC1G19DBVR, X2 32.768

Commit message: Trabajo dia 31 Oct. Update
SOLO TRABAJO SOBRE ESQUEMATICO.
- Inclusion pantalla 49".
- Cambio en el diseño de la gestion de la laimentacion. Inclusion de transistor P comandado por 2 N (Boton de encendido y Señal digital CPU)
- Multiplaxado del control del DCDC y del Switch de salida, entre las señales digitales de la CPU y el comparador.
- Se añaden fajas place holder.
Parts:
- removed C10, C12: 2.2uF, microbuilder:CAP_CERAMIC0805-NOOUTLINE
- removed C5: 100n, microbuilder:CAP_CERAMIC0603_NO
- removed GND, IOSENSE, ISENSE_RAW, RXI, RXI1, SCL_2, SDA_2, TST_MODE, TXO, TXO1, VBUS, VCC, VCC_2, VOUTSENSE: TESTPAD_TPSQB1,27, BeagleBone_Blue_R3:TESTPAD_TPSQB1,27
- removed J1: 2314820-6, connector 2x3-2mm:2314820-6
- removed K3: FLEX_CONN, Flex_3mm:FLEX4
- removed K4: FLEX6, Flex_3mm:FLEX6
- removed K5: FLEX8, Flex_3mm:FLEX8
- removed R45: 330, SparkFun-Resistors:RESISTOR0603
- removed TP48: TPTP08R, testpad:TPTP08R
- removed U2: TPS78230DDCR, TPS78230DDCR:TPS78230DDCR
- removed U5: MAX9062EUK+T, MAX9062:MAX9062EUK+T
- removed U7: MCP6071T-E/OT, MCP6071:MCP6071T-E/OT
- added C19: 100n, microbuilder:CAP_CERAMIC0603_NO
- added K2: FLEX6, Flex:FLEX6
- added Q1: BSS84W-7-F, BSS84W-7-F:BSS84W-7-F
- added Q2, Q3, Q5: 2N7002PW, SparkFun-DiscreteSemi:MOSFET-NCHANNEL2N7002PW
- added R48: 100R, SparkFun-Resistors:RESISTOR0603
- added R49: 10k, SparkFun-Resistors:RESISTOR0603
- added S1, S2, S3: PTS526_SKG15_SMTR2_LFS, PTS526_SKG15_SMTR2_LFS:PTS526_SKG15_SMTR2_LFS
- added U$30: 64X32_OLED_049, OLED 66 64x48:64X32_OLED_049
- C13: device microbuilder:CAP_CERAMIC0603_NO -> rcl:C-EUC0805
- C16, C17: value 1u -> 100n; device microbuilder:CAP_CERAMIC0603_NO -> rcl:C-EUC0805
- R1, R10, R14, R17, R2, R3, R4: device SparkFun-Resistors:RESISTOR0603 -> SparkFun-Resistors:RESISTOR0402
- R11: value 8.2k -> 8k2; device SparkFun-Resistors:RESISTOR0603 -> SparkFun-Resistors:RESISTOR0402
- R12: value 2.4k -> 2k2; device SparkFun-Resistors:RESISTOR0603 -> SparkFun-Resistors:RESISTOR0402
- R13: value 62k -> 100R; device SparkFun-Resistors:RESISTOR0603 -> SparkFun-Resistors:RESISTOR0402
- R15: value 2.4k -> 100R; device SparkFun-Resistors:RESISTOR0603 -> SparkFun-Resistors:RESISTOR0402
- R16: value 36k -> (none); device SparkFun-Resistors:RESISTOR0603 -> SparkFun-Resistors:RESISTOR0402
- R18: value RESISTOR0402 -> (none); device BeagleBone_Blue_R3:RESISTOR0402 -> SparkFun-Resistors:RESISTOR0402
- R5: value 100k -> (none); device SparkFun-Resistors:RESISTOR0603 -> SparkFun-Resistors:RESISTOR0402
- R6: value 10k -> (none); device SparkFun-Resistors:RESISTOR0603 -> SparkFun-Resistors:RESISTOR0402
- R7: value 10k -> 2k2; device SparkFun-Resistors:RESISTOR0603 -> SparkFun-Resistors:RESISTOR0402
- R8: value 120k -> 100R; device SparkFun-Resistors:RESISTOR0603 -> SparkFun-Resistors:RESISTOR0402
- R9: value 5.6k -> 2k2; device SparkFun-Resistors:RESISTOR0603 -> SparkFun-Resistors:RESISTOR0402
Connections:
- removed net #EN_DCDC: K5.P$8, U1.PA16/I2C/I0/SERCOM1+3.0
- removed net /FLAG_BATTLOW: R6.1, U1.PA19/I3/SERCOM1+3.3/I2SD0, U6.OUT
- removed net D+: U1.PA25/I13/SERCOM3+5.3/D+
- removed net D-: U1.PA24/I12/SERCOM3+5.2/D-
- removed net EN_VCC2: R5.2, U1.PA10/I10/AIN18/SERCOM0+2.2/I2SCK, U2.EN
- removed net FLAG_CHRG: R7.1, U1.PA15/I15/SERCOM3+4.3, U5.OUT
- removed net ISENSE_RAW: ISENSE_RAW.TP, K5.P$5, R12.2
- removed net N$11: R8.1, R9.1, U5.IN
- removed net N$12: U1.PA27/I15
- removed net N$14: U1.PA28/I8
- removed net N$15: TP48.TP, U1.PB03/I3/AIN11/SERCOM5.1
- removed net N$4: U1.PA06/EINT6/AIN6/SERCOM0.2
- removed net N$8: C17.1, R12.1, R13.2
- removed net OP_SWITCH: K5.P$4, U1.PA20/I4/SERCOM3+5.2/I2SSC
- removed net SCL2_CPU: R4.2, U1.PA17/I2C/I1/SERCOM1+3.1
- removed net SCL_2: K3.P$4, R1.1, R4.1, SCL_2.TP
- removed net SDA2_CPU: R3.2, U1.PA18/I2/SERCOM1+3.2
- removed net SDA_2: K3.P$1, R2.1, R3.1, SDA_2.TP
- removed net USB_SEL: U1.PA21/I5/SERCOM3+5.3/I2SFS0
- removed net VCC_2: C12.1, C13.1, C15.1, C5.1, K4.P$1, K5.P$2, U2.OUT, U7.VDD, U8.VCC, VCC_2.TP
- new net CPU_EN_OUT: R18.2, U1.PA16/I2C/I0/SERCOM1+3.0
- new net EN_OUT: K2.P$4, Q5.D, R18.1
- new net EN_VCC: Q3.G, R16.2, U1.PA10/I10/AIN18/SERCOM0+2.2/I2SCK
- new net IN_OVC: Q5.G, R48.2, R49.2
- new net N$2: C13.1, R8.2, R9.2, S1.COM_2
- new net N$3: C16.1, R12.2, R13.1, S2.COM_2
- new net N$58: R48.1, U6.OUT
- new net N$6: Q1.G, Q2.D, Q3.D, R5.2
- new net SCL_CPU: R4.2, U1.PA23/I2C/I7/SERCOM3+5.1/SOF
- new net SDA_CPU: R3.2, U1.PA22/I2C/I6/SERCOM3+5.0
- new net S_POWER: Q2.G, R15.2, R6.2
- net !RESET: now also K2.P$10; no longer J1.3
- net GND: now also C17.2, C19.2, K2.P$2, Q2.S, Q3.S, Q5.S, R16.1, R49.1, R6.1, S1.NO_2, S2.NO_2, S3.NO_2; no longer C10.2, C12.2, C5.2, GND.TP, J1.5, K3.P$2, K4.P$2, K5.P$3, R15.2, R5.1, R9.2, U2.GND, U5.GND, U5.GND_2, U7.VSS
- net IOSENSE: now also K2.P$8; no longer C17.2, IOSENSE.TP, R16.1, U7.VOUT
- net N$1: now also C17.1, R7.2, S3.COM_2; no longer R16.2, U7.VIN-
- net N$10: now also C19.1
- net N$13: now also C6.1, Q1.S, U3.EN, U3.IN; no longer C16.1, R13.1, U7.VIN+
- net N$19: no longer R45.1
- net N$22: no longer R45.2
- net RXI: now also K2.P$7; no longer RXI.TP, RXI1.TP
- net SCL: now also R1.1, R4.1; no longer K4.P$4, K5.P$6, U1.PA23/I2C/I7/SERCOM3+5.1/SOF
- net SDA: now also R2.1, R3.1; no longer K4.P$3, K5.P$1, U1.PA22/I2C/I6/SERCOM3+5.0
- net SWCLK: now also K2.P$6; no longer J1.4
- net SWDIO: now also K2.P$5; no longer J1.2
- net S_DOWN: now also R13.2; no longer K4.P$6
- net S_UP: now also R8.1; no longer K4.P$5
- net TST_MODE: no longer TST_MODE.TP
- net TXO: no longer TXO.TP, TXO1.TP
- net VBUS: now also K2.P$3, Q1.D, R5.1, R7.1; no longer C10.1, C6.1, K3.P$3, R8.2, U2.IN, U3.EN, U3.IN, VBUS.TP
- net VCC: now also C15.1, K2.P$1, R12.1, R9.1, U8.VCC; no longer J1.1, R6.2, R7.2, U5.VCC, VCC.TP
- net VOUTSENSE: now also K2.P$9; no longer K5.P$7, VOUTSENSE.TP
Other:
- note removed: "A VCC para que se pueda detectar cambios de voltaje en la bateria durante SLEEP"
- note removed: "A VCC para que se pueda detectar el pulsador de encendido que esta en la bateria"
- note removed: "Cortex Debug/ Program Connector"
- note removed: "FLEX BANDS"
- note removed: "G=16 BW=10Hz"
- note removed: "IOSENSE LOWPASS FILTERING"
- note removed: "TEST PADS"
- note removed: "Test pads are placed on the bottom for a bed of nails test setup. Ideally spacing between test pads should be greater or equal to 3mm"
- note removed: "VCC_2 -- POWER AND FILTERING"
- note removed: "Vtrigger=4.5V"
- moved on the sheet: BZ1, C13, C15, C16, C17, C18, C6, C7, C8, L7, R1, R10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

Commit message: Modificacion Ruteado CPU
Se añade la version 1 de las dimensiones del PCB y se posicionan los componentes sin ruteado.
FALTA: Circuito acondicionamiento Display .
Parts:
- removed Q2: 2N7002PW, SparkFun-DiscreteSemi:MOSFET-NCHANNEL2N7002PW
- removed R6: (no value), SparkFun-Resistors:RESISTOR0402
- R48: device SparkFun-Resistors:RESISTOR0603 -> SparkFun-Resistors:RESISTOR0402
- R49: value 10k -> 10K; device SparkFun-Resistors:RESISTOR0603 -> SparkFun-Resistors:RESISTOR0402
Connections:
- net CPU_EN_OUT renamed CPU_EN_DCDC
- net EN_OUT renamed EN_DCDC
- net EN_VCC renamed EN_VCC_2
- removed net N$13: C6.1, Q1.S, U3.EN, U3.IN
- new net N$4: U1.PA17/I2C/I1/SERCOM1+3.1
- new net OP_SWITCH: K2.P$11
- new net VCC_2: K2.P$12, Q1.S
- net GND: no longer Q2.S, R6.1
- net N$6: no longer Q2.D
- net S_POWER: no longer Q2.G, R6.2
- net VBUS: now also C6.1, U3.EN, U3.IN; no longer Q1.D, R5.1
- net VCC: now also Q1.D, R5.1
Other:
- moved on the sheet: C6, C7, C8, Q1, Q3, R14, R16, R17, R5, U3

Commit message: Update CPU PCB.
Routeado terminado v1. PENDIENTE DE REVISION.
Parts:
- added C10, C24, C25, C26, C5: 0.1uF, SparkFun-Capacitors:0.1UF-0402-16V-10%
- added C12, C23: 1.0uF, SparkFun-Capacitors:1.0UF-0402-16V-10%
- added C20: 2.2uF, SparkFun-Capacitors:2.2UF-0603-10V-20%
- added C21, C22: 4.7uF, SparkFun-Capacitors:4.7UF0603
- added Q2: BSS84W-7-F, BSS84W-7-F:BSS84W-7-F
- added Q4: 2N7002PW, SparkFun-DiscreteSemi:MOSFET-NCHANNEL2N7002PW
- added R6: 4K7, SparkFun-Resistors:RESISTOR0402
- added VBUS, VBUS1, VBUS2, VBUS3, VBUS4: TESTPAD_TPSQB1,27, BeagleBone_Blue_R3:TESTPAD_TPSQB1,27
- R1, R2: value 2k2 -> 4K7
- R3: value 100R -> 560K
- R4: value 100R -> (none)
Connections:
- removed net IN_OVC: Q5.G, R48.2, R49.2
- removed net SCL_CPU: R4.2, U1.PA23/I2C/I7/SERCOM3+5.1/SOF
- removed net SDA_CPU: R3.2, U1.PA22/I2C/I6/SERCOM3+5.0
- new net !RES: C24.1, R6.1, U$30.!RES
- new net C1N: C23.1, U$30.C1N
- new net C1P: C23.2, U$30.C1P
- new net C2N: C12.1, U$30.C2N
- new net C2P: C12.2, U$30.C2P
- new net IN_UVLO: Q5.G, R48.2, R49.2, U1.PA21/I5/SERCOM3+5.3/I2SFS0
- new net IREF: R3.2, U$30.IREF
- new net N$11: U1.PA25/I13/SERCOM3+5.3/D+
- new net N$12: U1.PA28/I8
- new net N$13: U1.PB03/I3/AIN11/SERCOM5.1
- new net N$14: U1.PA24/I12/SERCOM3+5.2/D-
- new net N$8: U1.PA27/I15
- new net VBAT_LCD: C25.1, Q2.S, U$30.VBAT
- new net VCOMH: C20.1, U$30.VCOMH
- new net VDD: C10.1, C22.1, R6.2, U$30.VDD
- new net VSS: U$30.VSS
- net EN_VCC_2: now also Q4.G
- net GND: now also C10.2, C20.2, C21.2, C22.2, C24.2, C25.2, C26.2, C5.2, Q4.S, R3.1
- net N$4: now also Q2.G, Q4.D, R4.2; no longer U1.PA17/I2C/I1/SERCOM1+3.1
- net OP_SWITCH: now also U1.PA17/I2C/I1/SERCOM1+3.1
- net SCL: now also U$30.SCL, U1.PA23/I2C/I7/SERCOM3+5.1/SOF; no longer R4.1
- net SDA: now also U$30.SDA, U1.PA22/I2C/I6/SERCOM3+5.0; no longer R3.1
- net VBUS: now also Q2.D, R4.1; no longer R7.1
- net VCC: now also C21.1, C5.1, R7.1, U$30.VCC; no longer C15.1, C18.1, R1.2, R2.2, U6.VCC, U8.VCC
- net VCC_2: now also C15.1, C18.1, C26.1, R1.2, R2.2, U6.VCC, U8.VCC
Other:
- moved on the sheet: R1, R2, R3, R4
