File: 02.Hardware/V1-ROVER-2K/Battery PCBs/BATT_DCDC/BATT_DCDC.sch (EAGLE design)
At the start: 54 parts, among them K3 FLEX8, Q1 NVTFS9D6P04M8LTAG, Q2 2N7002PW, Q5 2N7002PW, U1 MCP6071T-E/OT, U3 TPS55330RTET

Commit message: Update DCDC
Colocacion y Posicionamiento de los componentes en la tarjeta.
Pendiente de Routeado.
Parts:
- removed D1: BAT54S, BAT54S:BAT54S
- added C1, C4, C5: 10uF, SparkFun-Capacitors:10UF-0805-10V-10%
- added C18, C19: 47uF 25V, Wurth_Elektronik_Passive_Capacitors_rev19a:WCAP-CSGP_1210_885012109003
- added R10: 82k, SparkFun-Resistors:RESISTOR0402
- added R2: 20k, SparkFun-Resistors:RESISTOR0402
- added R3: 10k, SparkFun-Resistors:RESISTOR0402
- added R6: 5k1, SparkFun-Resistors:RESISTOR0402
- added R7: 680k, SparkFun-Resistors:RESISTOR0402
- added R8: 330k, SparkFun-Resistors:RESISTOR0402
- added R9: 160k, SparkFun-Resistors:RESISTOR0402
- added U7: TPIC2810D, EDCPSU - Rev2:TPIC2810D
- C20: value N.A. -> 47nF
- R11: value 5k1 -> 15k
- R12: value 8k2 -> 1k
- R13: value 169k -> 15k
- R14: value 39k -> 15k
- R15: value 120k -> 470k
- R40: value N.A. -> 78.7k
- R43: value 47k -> 78.7k
- RSENSE: value 100mR -> 10mR
Connections:
- new net N$10: R9.1, U7.DRAIN5
- new net N$11: R10.1, U7.DRAIN4
- new net N$2: R1.1, U7.DRAIN3
- new net N$3: R2.1, U7.DRAIN2
- new net N$5: R3.1, U7.DRAIN1
- new net N$6: R6.1, U7.DRAIN0
- new net N$7: R7.1, U7.DRAIN7
- new net N$9: R8.1, U7.DRAIN6
- net FB_TPS: now also R10.2, R2.2, R3.2, R6.2, R7.2, R8.2, R9.2
- net GND: now also C1.1, C18.1, C19.1, C4.1, C5.1, U7.!G, U7.A0, U7.A1, U7.A2, U7.GND; no longer D1.A, R1.1
- net SCL: now also U7.SCL
- net SDA: now also U7.SDA
- net VCC: now also C1.2, U7.VCC; no longer D1.K
- net VOUTSENSE: no longer D1.A/K
- net VSOURCE: now also C18.2, C19.2
- net VSYS: now also C4.2, C5.2
Other:
- note removed: "G= 1.62 Fcut = 1/R11*C2*2PI = 300 Hz"
- note removed: "ROVER 1K - v1"
- note removed: "vo/vi = 0.1875 3.0 v @ vi=16v"
- moved on the sheet: R1
