File: 02.HARDWARE/V2-ROVER-1K/01.PCB/PROG_BATT/PROG_BATT.sch (EAGLE design)
At the start: 19 parts, among them J1 302-S201, Q1 PJA3416AE_R1_00001, U3 ATE1D-5M3-10-Z

Commit message: Modificaciones y correcciones (WIP)
Parts:
- added C1: 100uF, SparkFun-Capacitors:100UF-POLAR-RADIAL-2.5MM-25V-20%
- added JP3: JUMPER-SMT_3_1-NC_PASTE_NO-SILK, SparkFun-Jumpers:JUMPER-SMT_3_1-NC_PASTE_NO-SILK
- added JP4: (no value), jumper:JP1E
Connections:
- removed net RXI: J2.TXO
- new net N$1: J2.DTR
- new net N$2: J2.RXI, JP3.1
- new net N$3: J2.TXO, JP3.3
- net GND: no longer C13.1
- net GND_PSU: now also C1.-, C13.1, JP4.2
- net TXO: now also JP3.2; no longer J2.RXI
- net VCC_PSU: now also C1.+, JP4.1
Other:
- note added: "ARM 20 pin std connector"
- note added: "Interruptor ON/OFF"
- moved on the sheet: D3, FUSE, JP2, R40, U3

Commit message: Correcion de letering pre-lanazdo
correcion de letras y Colocacion Pin Auxiliar TXO
Parts:
- added TXO1: (no value), SparkFun-Connectors:CONN_01POGOPIN_HOLE_LARGE
- renumbered VBUS10 to VBUS1, VBUS9 to VBUS
Connections:
- net TXO: now also TXO1.1
Changed lines of the file:
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@@
 <drawing>
 <settings>
-<setting alwaysvectorfont="no"/>
+<setting alwaysvectorfont="yes"/>
 <setting keepoldvectorfont="yes"/>
 <setting verticaltext="up"/>
@@
 </classes>
 <parts>
-<part name="VBUS9" library="SparkFun-Connectors" deviceset="CONN_01" device="POGOPIN_HOLE_LARGE"/>
+<part name="VBUS" library="SparkFun-Connectors" deviceset="CONN_01" device="POGOPIN_HOLE_LARGE"/>
 <part name="!RESET" library="SparkFun-Connectors" deviceset="CONN_01" device="POGOPIN_HOLE_LARGE"/>
 <part name="SWCLK" library="SparkFun-Connectors" deviceset="CONN_01" device="POGOPIN_HOLE_LARGE"/>
@@
 <part name="SWDIO" library="SparkFun-Connectors" deviceset="CONN_01" device="POGOPIN_HOLE_LARGE"/>
 <part name="GND" library="SparkFun-Connectors" deviceset="CONN_01" device="POGOPIN_HOLE_LARGE"/>
-<part name="VBUS10" library="SparkFun-Connectors" deviceset="CONN_01" device="POGOPIN_HOLE_LARGE"/>
+<part name="VBUS1" library="SparkFun-Connectors" deviceset="CONN_01" device="POGOPIN_HOLE_LARGE"/>
 <part name="J1" library="302-S201" deviceset="302-S201" device=""/>
 <part name="U3" library="ATE1D-5M3-10-Z" deviceset="ATE1D-5M3-10-Z" device=""/>
@@
 <part name="C1" library="SparkFun-Capacitors" library_urn="urn:adsk.eagle:library:510" deviceset="100UF-POLAR" device="-RADIAL-2.5MM-25V-20%" package3d_urn="urn:adsk.eagle:package:37415/1" value="100uF"/>
 <part name="JP3" library="SparkFun-Jumpers" library_urn="urn:adsk.eagle:library:528" deviceset="JUMPER-SMT_3_1-NC_PASTE" device="_NO-SILK" package3d_urn="urn:adsk.eagle:package:39291/1"/>
+<part name="TXO1" library="SparkFun-Connectors" deviceset="CONN_01" device="POGOPIN_HOLE_LARGE"/>
 </parts>
 <sheets>
@@
 </plain>
 <instances>
-<instance part="VBUS9" gate="G$1" x="119.38" y="256.54" smashed="yes">
+<instance part="VBUS" gate="G$1" x="119.38" y="256.54" smashed="yes">
 <attribute name="VALUE" x="116.84" y="251.714" size="1.778" layer="96" font="vector"/>
 <attribute name="NAME" x="116.84" y="259.588" size="1.778" layer="95" font="vector"/>
@@
 <attribute name="NAME" x="116.84" y="210.058" size="1.778" layer="95" font="vector"/>
 </instance>
-<instance part="VBUS10" gate="G$1" x="119.38" y="198.12" smashed="yes">
+<instance part="VBUS1" gate="G$1" x="119.38" y="198.12" smashed="yes">
 <attribute name="VALUE" x="116.84" y="193.294" size="1.778" layer="96" font="vector"/>
 <attribute name="NAME" x="116.84" y="201.168" size="1.778" layer="95" font="vector"/>
@@
 <attribute name="NAME" x="307.34" y="176.149" size="1.778" layer="95" font="vector" rot="R180"/>
 </instance>
+<instance part="TXO1" gate="G$1" x="119.38" y="181.61" smashed="yes">
+<attribute name="VALUE" x="116.84" y="176.784" size="1.778" layer="96" font="vector"/>
+<attribute name="NAME" x="116.84" y="184.658" size="1.778" layer="95" font="vector"/>
+</instance>
 </instances>
 <busses>
@@
 <net name="VBUS" class="0">
 <segment>
-<pinref part="VBUS9" gate="G$1" pin="1"/>
+<pinref part="VBUS" gate="G$1" pin="1"/>
 <wire x1="127" y1="256.54" x2="153.67" y2="256.54" width="0.1524" layer="91"/>
 <wire x1="153.67" y1="256.54" x2="153.67" y2="257.81" width="0.1524" layer="91"/>
@@
 </segment>
 <segment>
-<pinref part="VBUS10" gate="G$1" pin="1"/>
+<pinref part="VBUS1" gate="G$1" pin="1"/>
 <wire x1="127" y1="198.12" x2="153.67" y2="198.12" width="0.1524" layer="91"/>
 <label x="134.62" y="198.12" size="1.778" layer="95"/>
@@
 <label x="332.74" y="176.53" size="0.0508" layer="95" font="vector"/>
 </segment>
+<segment>
+<pinref part="TXO1" gate="G$1" pin="1"/>
+<wire x1="127" y1="181.61" x2="153.67" y2="181.61" width="0.1524" layer="91"/>
+<label x="134.62" y="181.61" size="1.778" layer="95"/>
+</segment>
 </net>
