File: 02.HARDWARE/V2-ROVER-1K/03.TESTBOARDS/TEST_CPU/TEST_CPU.brd (EAGLE design)
At the start: 93 x 100 mm, 48 parts, among them J2 302-S201, J3 DF40C-20DP-0.4V_51_, Q4 2N7002PW, Q5 2N7002PW, U1 MCP1825T-ADJE/DCSOT-223_5MC_M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, U3 ATE1D-5M3-10-Z

Commit message: TESTBOARDS Pedido PCBWAY 6ENERO
Revision antes de enviar a PCBWAY
Parts:
- added C1, C10, C11, C2, C8, C9: 100n, SparkFun-Capacitors:0805
- added JP1, JP2: JUMPER-SMT_2_NC_PASTE_SILK, SparkFun-Jumpers:SMT-JUMPER_2_NC_PASTE_SILK
- added R27, R28, R30: (no value), SparkFun-Resistors:0805
- moved D3 6.30 mm to (8.14, 71.1)
- moved R40 6.17 mm to (7.07, 65.8)
- moved R18 3.99 mm to (32.6, 71.5)
- moved R15 1.39 mm to (51.4, 83.0)
- moved R14 0.36 mm to (55.1, 79.8)
- moved C6 0.35 mm to (21.0, 80.0)
- moved R19 0.29 mm to (25.7, 78.3)
Connections:
- removed net GND2: U4.GND@7
- new net N$10: JP2.1, U4.GP0
- new net N$8: JP1.1, U4.GP1
- net ENABLE_LDO_ADJ: now also R27.2
- net GND: now also C1.2, C10.2, C11.2, C2.2, C8.2, C9.2, R27.1, R28.1, R30.1, U4.GND@7
- net N$27: now also R28.2
- net N$34: now also R30.2
- net RXI: now also JP2.2; no longer U4.GP0
- net TXO: now also JP1.2; no longer U4.GP1
- net VBUS: now also C1.1, C8.1
- net VCC: now also C10.1, C2.1, C9.1
- net VUSB: now also C11.1
Routing:
- net GND: track 148.1 -> 182.5 mm, vias 13 -> 15
- net VCC: track 34.7 -> 44.8 mm
- net VBUS: track 78.4 -> 86.2 mm
- net N$34: track 1.66 -> 8.25 mm
- net RXI: track 115.3 -> 109.1 mm
- net N$8: track 0.00 -> 5.86 mm
- net TXO: track 110.1 -> 104.3 mm
- net OP_SWITCH: track 85.3 -> 79.6 mm
- net N$10: track 0.00 -> 5.02 mm
- net ENABLE_LDO_ADJ: track 52.6 -> 56.9 mm
- net SW2: track 56.0 -> 52.4 mm
- net N$27: track 1.80 -> 4.63 mm
- net VBUSBAR: track 32.3 -> 34.8 mm
- net VUSB: track 71.2 -> 73.4 mm
- net FB_DAC: track 76.9 -> 76.0 mm
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Other:
- board text added: "T1"
- board text added: "T2"
- board text added: "T3"

Commit message: Cambio en la alimentacion del conector.
Cambio de Vcc en el conector de programacion a Vcc CPU.
Connections:
- net VCC: no longer J2.1
- net VCC_CPU: now also J2.1
Routing:
- net VCC_CPU: track 15.2 -> 47.1 mm
Changed lines of the file:
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@@
 <drawing>
 <settings>
-<setting alwaysvectorfont="no"/>
+<setting alwaysvectorfont="yes"/>
 <setting verticaltext="up"/>
 </settings>
@@
 <contactref element="DISPLAY" pad="2"/>
 <contactref element="R66" pad="1"/>
-<contactref element="J2" pad="1"/>
 <contactref element="U4" pad="3V3"/>
 <contactref element="J3" pad="6"/>
@@
 <wire x1="56.239996875" y1="89.42" x2="55.56" y2="89.42" width="0.508" layer="1"/>
 <wire x1="55.56" y1="89.42" x2="54.12" y2="90.86" width="0.508" layer="1"/>
+<wire x1="63.57" y1="42.98" x2="64.03" y2="89.42" width="0" layer="19" extent="1-1"/>
+<wire x1="69.99" y1="12.95" x2="68.61" y2="39.62" width="0" layer="19" extent="1-1"/>
+<wire x1="58.48" y1="13.17" x2="69.99" y2="12.95" width="0" layer="19" extent="1-1"/>
+<wire x1="81.94" y1="12.9" x2="69.99" y2="12.95" width="0" layer="19" extent="1-1"/>
+<wire x1="26.61" y1="42.46" x2="63.29" y2="39.5" width="0" layer="19" extent="1-1"/>
+<wire x1="23.78" y1="40.2" x2="23.78" y2="40.22" width="0" layer="19" extent="1-1"/>
+<wire x1="19.65" y1="53.13" x2="26.61" y2="42.46" width="0" layer="19" extent="1-1"/>
 </signal>
 <signal name="TEST_2">
@@
 <wire x1="49.14" y1="76.84" x2="50.14" y2="76.84" width="0.508" layer="1"/>
 <wire x1="50.14" y1="76.84" x2="50.3" y2="76.68" width="0.508" layer="1"/>
+<contactref element="J2" pad="1"/>
+<wire x1="40" y1="96" x2="40.75" y2="96" width="0.508" layer="16"/>
+<wire x1="39.75" y1="66.78" x2="39.69" y2="66.78" width="0.508" layer="16"/>
+<wire x1="40.75" y1="96" x2="42.52" y2="94.23" width="0.508" layer="16"/>
+<wire x1="42.52" y1="94.23" x2="42.52" y2="69.55" width="0.508" layer="16"/>
+<wire x1="42.52" y1="69.55" x2="39.75" y2="66.78" width="0.508" layer="16"/>
 </signal>
 <signal name="SWO">

Commit message: Pedido PCBWAY Enero - Revision de cambios de Javi
Se hacen cambios menores
Routing:
- net DSP_RST: track 19.2 -> 18.6 mm
- net GND: vias 15 -> 18
Other:
- outline, holes or cut-outs redrawn
- board text added: "GND"
