File: 02.HARDWARE/V2-ROVER-1K/03.TESTBOARDS/TEST_DCDC/TEST_DCDC.sch (EAGLE design)
At the start: 47 parts, among them J1 FEMALE 2x3, J2 OSTVN03A150, J3 OSTVN03A150, J4 OSTVN03A150, Q1 PJA3416AE_R1_00001, Q2 PJA3416AE_R1_00001, Q3 PJA3416AE_R1_00001, U3 ATE1D-5M3-10-Z, U6 AP62200WU-7

Commit message: wip previo a envio PCBWAY
Queda revisar todavia y rutear
Parts:
- added D1, D2, D4: 250mA/100V, SparkFun-DiscreteSemi:DIODE-BAS16J
Connections:
- removed net N$18: J3.2, Q2.D
- removed net N$26: J4.2, Q3.D
- removed net N$8: J2.2, Q1.D
- new net N$1: D4.A, J4.3, Q3.D
- new net N$21: D1.A, J2.3, Q1.D
- new net N$3: D2.A, J3.3, Q2.D
- net VOUT+: now also D1.C, D2.C, D4.C
- net VOUT-: no longer J2.3, J3.3, J4.3
Other:
- note added: "test DCDC v1-Ene23"
- note removed: "Carrier Motor Driver v1-Sep22"
- moved on the sheet: J2, J3, J4, Q1, Q2, Q3, R11, R12, R13, R14, R15, R16

Commit message: Version 1 pendiente de revision
Parts:
- removed C14, C15, C16, C17: (no value), rcl:C-EUC0805
- removed ENA: TESTPAD_TPSQPAD1-17, BeagleBone_Blue_R3:TESTPAD_TPSQPAD1-17
- removed L1: SRN8040-8R2Y, SRN8040-8R2Y:SRN8040-8R2Y
- removed R38, R39: 10K, SparkFun:RESISTOR0805-RES
- removed U6: AP62200WU-7, AP62200WU-7:AP62200WU-7
- added C1, C2: 100n, rcl:C-EUC0805
- added D5: (no value), SparkFun-LED:LED3MM
- added J5: ACJS-MHDR, ACJSMHDR:ACJS-MHDR
- added J6, J7, J8, J9: (no value), SparkFun-Connectors:CONN_02
- added JP1: JUMPER-SMT_3_1-NC_PASTE_SILK, SparkFun-Jumpers:JUMPER-SMT_3_1-NC_PASTE_SILK
- added Q4: 310mA/60V/1.6Ω, SparkFun-DiscreteSemi:MOSFET-NCH-2N7002PW
- added R1: (no value), SparkFun-Resistors:RESISTOR0805
- added R2, R3: 10K, SparkFun-Resistors:RESISTOR0805
- added R4: 10K, SparkFun:RESISTOR0805-RES
- added U1: MCP4725, SparkFun-IC-Conversion:MCP4725SOT-23
Connections:
- removed net EN_LDO: ENA.TP, U6.EN
- removed net N$23: U4.GP9
- removed net N$31: C14.2, U6.BST
- removed net N$32: C14.1, L1.1, U6.SW
- removed net N$33: R38.1, R39.2, U6.FB
- removed net TEST_4: U4.GP20
- removed net TEST_5: U4.GP15
- removed net VBUSBAR: C17.1, D3.A, U3.1, U6.VIN
- removed net VCC_PSU: C13.2, U3.2
- new net FB_DAC_PWM: JP1.3, U4.GP11
- new net N$18: JP1.1, U1.VOUT
- new net N$26: D5.C, R4.2
- new net N$27: D5.A, U4.VBUS
- new net OP_SWITCH_CPU: Q4.G, U4.GP10
- new net VBUS: D3.A, U3.1, Z1.K
- new net VBUS_PSU: C13.2, J6.1, J6.2, U3.2
- net DSP_RST: now also U4.GP12
- net EN_DCDC: now also U4.GP9; no longer U4.GP11
- net FB_DAC: now also JP1.2; no longer U4.GP12
- net GND: now also C1.1, C2.1, J7.1, J7.2, Q4.S, R4.1, U1.AO, U1.VSS; no longer C15.1, C16.1, C17.2, R39.1, U6.GND
- net IOSENSE: now also U4.GP28_A2; no longer U4.GP27_A1
- net OP_SWITCH: now also Q4.D, R1.1; no longer U4.GP10
- net R1: now also U4.GP22; no longer U4.GP7
- net R2: now also U4.GP21; no longer U4.GP13
- net R3: now also U4.GP20; no longer U4.GP14
- net SCL: now also R2.1, U1.SCL
- net SDA: now also R3.1, U1.SDA
- net TEST_1: now also U4.GP15; no longer U4.GP26_A0
- net TEST_2: now also U4.GP14; no longer U4.GP22
- net TEST_3: now also U4.GP13; no longer U4.GP21
- net VCC: now also C1.2, C2.2, R1.2, R2.2, R3.2, U1.VDD, U4.3V3; no longer C15.2, C16.2, L1.2, R38.2, U4.VBUS, Z1.K
- net VOUT+: now also J5.6, J8.1, J8.2
- net VOUT-: now also J5.1, J5.4, J5.5, J9.1, J9.2
- net VOUTSENSE: now also U4.GP27_A1; no longer U4.GP28_A2
Other:
- note added: "CONNECTOR TO DUT"
- note added: "DAC"
- note added: "JACK OUTPUT"
- note added: "Test.DCDC Rover R1 v1-Ene23"
- note added: "VBUS OUTPUT"
- note removed: "3V3 DCDC CONVERTER"
- note removed: "test DCDC v1-Ene23"
- moved on the sheet: C13, C3, C4, C5, D1, D2, D3, D4, J2, J3, J4, Q1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

Commit message: Pedido PCBWAY ene-23 - revision despues de diseño
Parts:
- added C6: 10uF, Wurth_Elektronik_Passive_Capacitors_rev19a:WCAP-CSGP_1206_885012008001
- added R17: 33k, SparkFun-Resistors:RESISTOR0805
Connections:
- net N$1 renamed R2_OUT
- net N$21 renamed R1_OUT
- net N$3 renamed R3_OUT
- net GND: now also C6.1, R17.1
- net OP_SWITCH_CPU: now also R17.2
- net VCC: now also C6.2
Other:
- moved on the sheet: D2, D4, J3, J4, Q2, Q3, R13, R14, R15, R16
