File: 02.HARDWARE/V2-ROVER R-1/03.TESTBOARDS/CIRULO_PANEL/CIRULO_PANEL.brd (EAGLE design)
At the start: 43 x 57.3 mm, 13 parts, among them J1 302-S201, Q1 PJA3416AE_R1_00001, U3 ATE1D-5M3-10-Z

Commit message: Asignacion de Valores a los componentes pasivos de las tarjetas de Testeo. Actualziacion de las BOMs.
Parts:
- C13: value (none) -> 100n
- R40: value 10K -> 220
Changed lines of the file:
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@@
 <attribute name="NAME" x="56.1638" y="71.9366" size="1.27" layer="28" ratio="6" rot="SMR270"/>
 </element>
-<element name="C13" library="rcl" library_urn="urn:adsk.eagle:library:334" package="C0805" package3d_urn="urn:adsk.eagle:package:23617/2" value="" x="50.56" y="75.94" smashed="yes" rot="MR180">
+<element name="C13" library="rcl" library_urn="urn:adsk.eagle:library:334" package="C0805" package3d_urn="urn:adsk.eagle:package:23617/2" value="100n" x="50.56" y="75.94" smashed="yes" rot="MR180">
 <attribute name="NAME" x="50.59" y="74.37" size="0.6096" layer="26" rot="MR180" align="center"/>
 <attribute name="POPULARITY" value="88" x="45.56" y="75.94" size="1.778" layer="28" rot="MR180" display="off"/>
@@
 <attribute name="VALUE" x="37.054" y="75.24" size="0.6096" layer="28" font="vector" ratio="20" rot="MR90" align="top-center"/>
 </element>
-<element name="R40" library="SparkFun" package="0805" value="10K" x="44.97" y="78.14" smashed="yes" rot="MR0">
+<element name="R40" library="SparkFun" package="0805" value="220" x="44.97" y="78.14" smashed="yes" rot="MR0">
 <attribute name="NAME" x="44.832" y="79.2655" size="0.6096" layer="26" rot="MR0" align="center"/>
 <attribute name="VALUE" x="45.986" y="76.743" size="0.4064" layer="28" rot="MR0"/>
