File: 02.HARDWARE/V2-ROVER R-1/01.PCB/BATT_PCB_JACK/PCB_JACK.sch (EAGLE design)
At the start: 2 parts

Commit message: Connector Jack
Parts:
- removed PAD1, PAD2: WIREPADSMD2,54-5,08, wirepad:WIREPADSMD2,54-5,08
Connections:
- removed net GND: PAD1.P
- removed net VCC: PAD2.P
Changed lines of the file:
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@@
 </classes>
 <parts>
-<part name="PAD1" library="wirepad" library_urn="urn:adsk.eagle:library:412" deviceset="WIREPAD" device="SMD2,54-5,08" package3d_urn="urn:adsk.eagle:package:30841/1"/>
-<part name="PAD2" library="wirepad" library_urn="urn:adsk.eagle:library:412" deviceset="WIREPAD" device="SMD2,54-5,08" package3d_urn="urn:adsk.eagle:package:30841/1"/>
 </parts>
 <sheets>
@@
 </plain>
 <instances>
-<instance part="PAD1" gate="G$1" x="66.04" y="20.32" smashed="yes">
-<attribute name="NAME" x="64.897" y="22.1742" size="1.778" layer="95"/>
-<attribute name="VALUE" x="64.897" y="17.018" size="1.778" layer="96"/>
-</instance>
-<instance part="PAD2" gate="G$1" x="55.88" y="5.08" smashed="yes">
-<attribute name="NAME" x="54.737" y="6.9342" size="1.778" layer="95"/>
-<attribute name="VALUE" x="54.737" y="1.778" size="1.778" layer="96"/>
-</instance>
 </instances>
 <busses>
@@
 <wire x1="68.58" y1="20.32" x2="93.98" y2="20.32" width="0.1524" layer="91"/>
 <label x="76.2" y="20.32" size="1.778" layer="95"/>
-<pinref part="PAD1" gate="G$1" pin="P"/>
 </segment>
 </net>
@@
 <wire x1="58.42" y1="5.08" x2="91.44" y2="5.08" width="0.1524" layer="91"/>
 <label x="71.12" y="5.08" size="1.778" layer="95"/>
-<pinref part="PAD2" gate="G$1" pin="P"/>
 </segment>
 </net>
@@
 </schematic>
 </drawing>
-<compatibility>
-<note version="8.2" severity="warning">
-Since Version 8.2, EAGLE supports online libraries. The ids
-of those online libraries will not be understood (or retained)
-with this version.
-</note>
-<note version="8.3" severity="warning">
-Since Version 8.3, EAGLE supports URNs for individual library
-assets (packages, symbols, and devices). The URNs of those assets
-will not be understood (or retained) with this version.
-</note>
-<note version="8.3" severity="warning">
-Since Version 8.3, EAGLE supports the association of 3D packages
-with devices in libraries, schematics, and board files. Those 3D
-packages will not be understood (or retained) with this version.
-</note>
-</compatibility>
 </eagle>
