File: 02.HARDWARE/V2-ROVER R-1/01.PCB/BATT_CONNECTOR - INVERSOR/HISTORY/V2/BATT_CONNECTOR.sch (EAGLE design)
At the start: 7 parts, among them IC1 AP7370-50W5-7

Commit message: Diseño Dan Kubin version inicial
Parts:
- removed C1, C2: 1.0uF, SparkFun-Capacitors:1.0UF-0805-25V-(+80/-20%)
- removed IC1: AP7370-50W5-7, AP7370-50W5-7:AP7370-50W5-7
- removed LED1: 150080GS75000, 150080GS75000:150080GS75000
- removed N, P: TPSQTP20SQ, testpad:TPSQTP20SQ
- removed R1: (no value), SparkFun-Resistors:RESISTOR0805
- added !RESET, GND, RXI, SWCLK, SWDIO, TXO, VO+, VO-, VOUT+1, VOUT-1: TPB2,54, testpad:TPB2,54
- added D1: SM2T18A, SM2T18A:SM2T18A
- added H1, H2: S1761-42R, S1761-42R:S1761-42R
- added K1: FLEX11, Flex_3mm:FLEX11
- added Q1: SSM3J338R,LF, SSM3J338R_LF:SSM3J338R,LF
Connections:
- removed net N$11: C2.1, IC1.VOUT, R1.1
- removed net N$12: LED1.A, R1.2
- removed net VIN: C1.1, IC1.VIN, P.TP
- new net !RESET: !RESET.TP, K1.P$9
- new net RXI: K1.P$8, RXI.TP
- new net SWCLK: K1.P$7, SWCLK.TP
- new net SWDIO: K1.P$5, SWDIO.TP
- new net TXO: K1.P$6, TXO.TP
- new net VBUS: K1.P$1, K1.P$2, Q1.S
- new net VBUS_IN: H1.1, H2.1, Q1.D
- new net VOUT+: D1.K, K1.P$11, VO+.TP, VOUT+1.TP
- new net VOUT-: D1.A, K1.P$10, VO-.TP, VOUT-1.TP
- net GND: now also GND.TP, K1.P$3, K1.P$4, Q1.G; no longer C1.2, C2.2, IC1.GND, LED1.K, N.TP
