File: 02.HARDWARE/V2-ROVER R-1/01.PCB/BATT_DCDC/BATT_DCDC.brd (EAGLE design)
At the start: 20.4 x 34.4 mm, 67 parts, among them J1 DF40C-20DP-0.4V_51_, K1 FLEX11, Q1 NVTFS9D6P04M8LTAG, Q2 2N7002PW, Q3 PMV20XNER, U1 MCP6071T-E/OT, U2 LM5114BMF_NOPB, U3 TPS55330RTET, U7 MCP6071T-E/OT

Commit message: Adiccion de Fiducidiales y actualizacion de Version
Other:
- board text added: "BATT_DCDC ROVER R-1 Nov'23 v5"
- board text removed: "BATT_DCDC ROVER R-1 v4-SEP'23"
Changed lines of the file:
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@@
 <drawing>
 <settings>
-<setting alwaysvectorfont="yes"/>
+<setting alwaysvectorfont="no"/>
 <setting keepoldvectorfont="yes"/>
 <setting verticaltext="up"/>
@@
 <text x="67.91" y="5.05" size="0.6096" layer="26" font="vector" rot="MR180" align="center">BATT_DCDC
 ROVER R-1
-v4-SEP'23</text>
+Nov'23 v5</text>
 <circle x="67.69" y="35.12" radius="0.9" width="0.1" layer="20"/>
 <circle x="58.94" y="10.62" radius="0.9" width="0.1" layer="20"/>
