File: 02.HARDWARE/V2-ROVER R-1/01.PCB/BATT_FLEX11/BATT_FLEX11.sch (EAGLE design)
At the start: 4 parts, among them K3 FLEX11, K4 FLEX11, K7 FLEX11, K8 FLEX11

Commit message: Nomenclatura de versiones
Other:
- note added: "FLEX_11 v1_Ene'23"
Changed lines of the file:
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@@
 <drawing>
 <settings>
-<setting alwaysvectorfont="yes"/>
+<setting alwaysvectorfont="no"/>
 <setting verticaltext="up"/>
 </settings>
@@
 <sheet>
 <plain>
+<text x="101.6" y="123.19" size="5.08" layer="91">FLEX_11
+v1_Ene'23</text>
 </plain>
 <instances>
@@
 </schematic>
 </drawing>
+<compatibility>
+<note version="6.3" minversion="6.2.2" severity="warning">
+Since Version 6.2.2 text objects can contain more than one line,
+which will not be processed correctly with this version.
+</note>
+</compatibility>
 </eagle>
