File: 02.HARDWARE/V3-Rover Venus/01-PCB/CRADLE/cradle_venus.brd (EAGLE design)
At the start: 54.7 x 69.2 mm, 30 parts, among them IC1 MCP73831T-2ACI_OT, IC2 WS2812B, IC3 ATTINY1616-SNR, IC4 WS2812B, IC5 WS2812B, IC6 WS2812B, IC7 WS2812B, IC8 WS2812B, J1 DX07S016JA1R1500, Q5 DMG3415U-7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

Commit message: Cradle Venus
Parts:
- C3, C4: value (none) -> 100n
- R20: value (none) -> 100R
- R21: value (none) -> 100K
Changed lines of the file:
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@@
 <drawing>
 <settings>
-<setting alwaysvectorfont="yes"/>
+<setting alwaysvectorfont="no"/>
 <setting verticaltext="up"/>
 </settings>
@@
 <attribute name="VALUE" x="113.4" y="62.691" size="0.6096" layer="27" font="vector" ratio="20" align="top-center"/>
 </element>
-<element name="R20" library="SparkFun-Resistors" library_urn="urn:adsk.eagle:library:532" package="0805" package3d_urn="urn:adsk.eagle:package:39651/1" value=" " x="114.13" y="31.5" smashed="yes" rot="R90">
+<element name="R20" library="SparkFun-Resistors" library_urn="urn:adsk.eagle:library:532" package="0805" package3d_urn="urn:adsk.eagle:package:39651/1" value="100R" x="114.13" y="31.5" smashed="yes" rot="R90">
 <attribute name="NAME" x="114.15" y="34.001" size="0.8128" layer="25" font="vector" ratio="10" rot="R180" align="bottom-center"/>
 <attribute name="PROD_ID" value=" " x="156.04" y="46.74" size="1.778" layer="27" rot="R90" display="off"/>
 <attribute name="VALUE" x="115.019" y="31.5" size="0.6096" layer="27" font="vector" ratio="20" rot="R90" align="top-center"/>
 </element>
-<element name="R21" library="SparkFun-Resistors" library_urn="urn:adsk.eagle:library:532" package="0805" package3d_urn="urn:adsk.eagle:package:39651/1" value=" " x="118.3" y="29.51" smashed="yes" rot="R180">
+<element name="R21" library="SparkFun-Resistors" library_urn="urn:adsk.eagle:library:532" package="0805" package3d_urn="urn:adsk.eagle:package:39651/1" value="100K" x="118.3" y="29.51" smashed="yes" rot="R180">
 <attribute name="NAME" x="118.3" y="28.621" size="0.8128" layer="25" font="vector" ratio="10" rot="R180" align="bottom-center"/>
 <attribute name="PROD_ID" value=" " x="99.25" y="71.42" size="1.778" layer="27" rot="R180" display="off"/>
@@
 <attribute name="VALUE" x="94.45" y="71.417" size="0.6096" layer="27" font="vector" ratio="20" align="top-center"/>
 </element>
-<element name="C3" library="resistor" library_urn="urn:adsk.eagle:library:348" package="C0805" package3d_urn="urn:adsk.eagle:package:23617/2" value="" x="104.33" y="70.79" smashed="yes">
+<element name="C3" library="resistor" library_urn="urn:adsk.eagle:library:348" package="C0805" package3d_urn="urn:adsk.eagle:package:23617/2" value="100n" x="104.33" y="70.79" smashed="yes">
 <attribute name="NAME" x="103.06" y="72.06" size="0.8128" layer="25" font="vector"/>
 <attribute name="VALUE" x="103.06" y="68.25" size="1.27" layer="27"/>
 </element>
-<element name="C4" library="resistor" library_urn="urn:adsk.eagle:library:348" package="C0805" package3d_urn="urn:adsk.eagle:package:23617/2" value="" x="92.06" y="40.7" smashed="yes" rot="R270">
+<element name="C4" library="resistor" library_urn="urn:adsk.eagle:library:348" package="C0805" package3d_urn="urn:adsk.eagle:package:23617/2" value="100n" x="92.06" y="40.7" smashed="yes" rot="R270">
 <attribute name="NAME" x="90.84" y="42.89" size="0.8128" layer="25" font="vector"/>
 <attribute name="VALUE" x="89.52" y="41.97" size="1.27" layer="27" rot="R270"/>
